Commit message: Remove some warnings

File: record_trajectory/urdf/robot.xacro (robot description, xacro)
@@ -1,12 +1,7 @@
 <?xml version="1.0" ?>
-<robot name="robot" xmlns:xacro="http://ros.org/wiki/xacro">
+<robot name="ur5" xmlns:xacro="http://ros.org/wiki/xacro">
   <xacro:include filename="$(find ur_description)/urdf/common.gazebo.xacro" />
   <xacro:include filename="$(find ur_description)/urdf/ur5.urdf.xacro" />
   <xacro:ur5_robot prefix="" joint_limited="false"/>
-  <link name="world" />
-  <joint name="world_joint" type="fixed">
-    <parent link="world" />
-    <child link = "base_link" />
-  </joint>
   <link name="camera">
     <visual>
